File: env/env.sch (EAGLE design)
At the start: 90 parts, among them IC1 DG403DJD, IC2 OPA4130U, IC3 4001D, IC4 OPA2134D, IC5 OPA4130U, Q1 BC847ALT1SMD, Q2 BC857ALT1SMD, X1 2516-

Commit message: added leds to env
Parts:
- added D1: (no value), dan:DUOLED5MM
- added LED1, LED2: (no value), dan:LED5MM
- added R46, R47, R48: 10k, dan:R-US_R0603
Connections:
- new net N$43: LED2.C, R46.2
- new net N$52: D1.AG, D1.AR, R48.1
- new net N$53: LED1.C, R47.2
- net GND: now also R46.1, R47.1, R48.2
- net N$2: now also LED2.A
- net N$36: now also D1.C
- net N$9: now also LED1.A
Changed lines of the file:
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@@
 <part name="C20" library="dan" deviceset="C-US" device="C0603" value="1u"/>
 <part name="C21" library="dan" deviceset="C-US" device="C0603" value="1u"/>
+<part name="D1" library="dan" deviceset="DUOLED5MM" device=""/>
+<part name="LED1" library="dan" deviceset="LED" device="5MM"/>
+<part name="LED2" library="dan" deviceset="LED" device="5MM"/>
+<part name="R46" library="dan" deviceset="R-US_" device="R0603" value="10k"/>
+<part name="R47" library="dan" deviceset="R-US_" device="R0603" value="10k"/>
+<part name="GND28" library="dan" deviceset="GND" device=""/>
+<part name="GND29" library="dan" deviceset="GND" device=""/>
+<part name="R48" library="dan" deviceset="R-US_" device="R0603" value="10k"/>
+<part name="GND30" library="dan" deviceset="GND" device=""/>
 </parts>
 <sheets>
@@
 <instance part="C20" gate="G$1" x="-111.76" y="27.94" rot="R180"/>
 <instance part="C21" gate="G$1" x="-119.38" y="43.18"/>
+<instance part="D1" gate="1" x="220.98" y="30.48" rot="R270"/>
+<instance part="LED1" gate="G$1" x="127" y="66.04"/>
+<instance part="LED2" gate="G$1" x="43.18" y="17.78"/>
+<instance part="R46" gate="G$1" x="43.18" y="5.08" rot="R90"/>
+<instance part="R47" gate="G$1" x="127" y="50.8" rot="R90"/>
+<instance part="GND28" gate="1" x="127" y="38.1"/>
+<instance part="GND29" gate="1" x="43.18" y="-5.08"/>
+<instance part="R48" gate="G$1" x="220.98" y="12.7" rot="R270"/>
+<instance part="GND30" gate="1" x="220.98" y="2.54"/>
 </instances>
 <busses>
@@
 <wire x1="30.48" y1="33.02" x2="35.56" y2="33.02" width="0.1524" layer="91"/>
 <junction x="27.94" y="58.42"/>
+<wire x1="43.18" y1="25.4" x2="30.48" y2="25.4" width="0.1524" layer="91"/>
+<wire x1="30.48" y1="25.4" x2="30.48" y2="33.02" width="0.1524" layer="91"/>
+<junction x="30.48" y="33.02"/>
+<pinref part="LED2" gate="G$1" pin="A"/>
+<wire x1="43.18" y1="20.32" x2="43.18" y2="25.4" width="0.1524" layer="91"/>
 </segment>
 </net>
@@
 <wire x1="-27.94" y1="27.94" x2="-27.94" y2="30.48" width="0.1524" layer="91"/>
 </segment>
+<segment>
+<pinref part="GND30" gate="1" pin="GND"/>
+<pinref part="R48" gate="G$1" pin="2"/>
+<wire x1="220.98" y1="5.08" x2="220.98" y2="7.62" width="0.1524" layer="91"/>
+</segment>
+<segment>
+<pinref part="GND28" gate="1" pin="GND"/>
+<pinref part="R47" gate="G$1" pin="1"/>
+<wire x1="127" y1="40.64" x2="127" y2="45.72" width="0.1524" layer="91"/>
+</segment>
+<segment>
+<pinref part="R46" gate="G$1" pin="1"/>
+<pinref part="GND29" gate="1" pin="GND"/>
+<wire x1="43.18" y1="0" x2="43.18" y2="-2.54" width="0.1524" layer="91"/>
+</segment>
 </net>
 <net name="N$3" class="0">
@@
 <pinref part="IC2" gate="B" pin="OUT"/>
 <wire x1="116.84" y1="66.04" x2="119.38" y2="66.04" width="0.1524" layer="91"/>
-<wire x1="119.38" y1="66.04" x2="119.38" y2="83.82" width="0.1524" layer="91"/>
+<wire x1="119.38" y1="66.04" x2="119.38" y2="73.66" width="0.1524" layer="91"/>
 <pinref part="R7" gate="G$1" pin="1"/>
+<wire x1="119.38" y1="73.66" x2="119.38" y2="83.82" width="0.1524" layer="91"/>
 <wire x1="119.38" y1="83.82" x2="119.38" y2="114.3" width="0.1524" layer="91"/>
 <wire x1="119.38" y1="114.3" x2="109.22" y2="114.3" width="0.1524" layer="91"/>
@@
 <wire x1="121.92" y1="83.82" x2="119.38" y2="83.82" width="0.1524" layer="91"/>
 <junction x="119.38" y="83.82"/>
+<pinref part="LED1" gate="G$1" pin="A"/>
+<wire x1="127" y1="68.58" x2="127" y2="73.66" width="0.1524" layer="91"/>
+<wire x1="127" y1="73.66" x2="119.38" y2="73.66" width="0.1524" layer="91"/>
+<junction x="119.38" y="73.66"/>
 </segment>
 </net>
@@
 <wire x1="223.52" y1="45.72" x2="220.98" y2="45.72" width="0.1524" layer="91"/>
 <junction x="220.98" y="45.72"/>
+<pinref part="D1" gate="1" pin="C"/>
+<wire x1="220.98" y1="33.02" x2="220.98" y2="45.72" width="0.1524" layer="91"/>
 </segment>
 </net>
@@
 </segment>
 </net>
+<net name="N$52" class="0">
+<segment>
+<pinref part="D1" gate="1" pin="AG"/>
+<wire x1="213.36" y1="30.48" x2="208.28" y2="30.48" width="0.1524" layer="91"/>
+<wire x1="208.28" y1="30.48" x2="208.28" y2="20.32" width="0.1524" layer="91"/>
+<wire x1="208.28" y1="20.32" x2="220.98" y2="20.32" width="0.1524" layer="91"/>
+<wire x1="220.98" y1="20.32" x2="231.14" y2="20.32" width="0.1524" layer="91"/>
+<wire x1="231.14" y1="20.32" x2="231.14" y2="30.48" width="0.1524" layer="91"/>
+<pinref part="D1" gate="1" pin="AR"/>
+<wire x1="231.14" y1="30.48" x2="228.6" y2="30.48" width="0.1524" layer="91"/>
+<pinref part="R48" gate="G$1" pin="1"/>
+<wire x1="220.98" y1="17.78" x2="220.98" y2="20.32" width="0.1524" layer="91"/>
+<junction x="220.98" y="20.32"/>
+</segment>
+</net>
+<net name="N$53" class="0">
+<segment>
+<pinref part="R47" gate="G$1" pin="2"/>
+<pinref part="LED1" gate="G$1" pin="C"/>
+<wire x1="127" y1="55.88" x2="127" y2="60.96" width="0.1524" layer="91"/>
+</segment>
+</net>
+<net name="N$43" class="0">
+<segment>
+<pinref part="LED2" gate="G$1" pin="C"/>
+<pinref part="R46" gate="G$1" pin="2"/>
+<wire x1="43.18" y1="12.7" x2="43.18" y2="10.16" width="0.1524" layer="91"/>
+</segment>
+</net>

Commit message: did some post fab changes to env
Parts:
- R14: value 1k -> 10k
Other:
- note added: "+in should be 6V"
- note added: "Attach this 6V to VL on dg403"
- note added: "Changed to 10k"
- note added: "Polarity backwards"
Changed lines of the file:
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@@
 <part name="Q1" library="dan" deviceset="BC847*" device="SMD" technology="ALT1"/>
 <part name="Q2" library="dan" deviceset="BC857*" device="SMD" technology="ALT1"/>
-<part name="R14" library="dan" deviceset="R-US_" device="R0603" value="1k"/>
+<part name="R14" library="dan" deviceset="R-US_" device="R0603" value="10k"/>
 <part name="R15" library="dan" deviceset="R-US_" device="R0603" value="90"/>
 <part name="R16" library="dan" deviceset="R-US_" device="R0603" value="2.1k"/>
@@
 <text x="-38.1" y="20.32" size="1.778" layer="91">Check these</text>
 <text x="-48.26" y="121.92" size="1.778" layer="91">Add LEDs!!!!</text>
+<text x="71.12" y="53.34" size="1.778" layer="91">+in should be 6V </text>
+<text x="86.36" y="-35.56" size="1.778" layer="91">Changed to 10k</text>
+<text x="137.16" y="101.6" size="1.778" layer="91">Attach this 6V to VL on dg403</text>
+<text x="0" y="-5.08" size="1.778" layer="91">Polarity backwards</text>
+<text x="10.16" y="-83.82" size="1.778" layer="91">Polarity backwards</text>
+<text x="116.84" y="-33.02" size="1.778" layer="91">Polarity backwards</text>
+<text x="134.62" y="38.1" size="1.778" layer="91">Polarity backwards</text>
+<text x="172.72" y="93.98" size="1.778" layer="91">Polarity backwards</text>
 </plain>
 <instances>

Commit message: made changes to env to send out again.  need to fix bi color led.
Parts:
- added Q3, Q4: BC847ALT1SMD, dan:BC847ALT1SMD
- added R49, R50, R52: 10K, dan:R-US_R0603
- added R51, R53: 1K, dan:R-US_R0603
- R10: value 1k -> 500
- R12: value 10k -> 4.7k
Connections:
- removed net N$40 (its old number): OS.E, R38.1
- new net N$14: ADAR.S, Q4.C, R52.2
- new net N$37: OS.A, R38.1
- new net N$51: Q3.B, R10.2, R49.1
- new net N$54: IC1A.IN, R51.1, R7.2
- new net N$56: Q4.B, R53.1
- net +12V: now also Q3.C, R52.1
- net -12V: now also R50.2
- net ENV: now also ASHAPE.A; no longer ASHAPE.E
- net GND: now also ACVA.A, ASHAPE.E, Q4.E, R49.2; no longer ACVA.E, ASHAPE.A, IC2A.+IN
- net N$11: now also Q3.E, R50.1, R51.2; no longer IC1A.IN, R10.2, R7.2
- net N$13: now also IC2A.+IN
- net N$16: now also IC2D.+IN; no longer IC2D.-IN
- net N$17: now also IC2D.-IN; no longer IC2D.+IN
- net N$20: now also R53.2; no longer ADAR.S
- net N$28: now also R32.1; no longer R31.2
- net N$30: now also R31.2; no longer R32.1
- net N$38: now also ACVA.E; no longer ACVA.A
- net N$39: now also OS.E; no longer OS.A
Other:
- note removed: "+in should be 6V"
- note removed: "Attach this 6V to VL on dg403"
- moved on the sheet: A, ACVA, ADAR, ASHAPE, AUV, C1, C10, C11, C12, C13, C14, C15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

Commit message: got the 2nd set of gerbers for env ready to send out
Parts:
- removed D1: (no value), dan:DUOLED5MM
- added LED3: (no value), dan:LED5MM
- R9: value 10k -> 4.7k
Connections:
- removed net N$52: D1.AG, D1.AR, R48.1
- new net N$57: LED3.C, R48.1
- net N$36: now also LED3.A; no longer D1.C
Other:
- note added: "bicolor"
- note removed: "Add LEDs!!!!"
- note removed: "This is not confirmed."
Changed lines of the file:
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@@
 <part name="R7" library="dan" deviceset="R-US_" device="R0603" value="1k"/>
 <part name="R8" library="dan" deviceset="R-US_" device="R0603" value="10k"/>
-<part name="R9" library="dan" deviceset="R-US_" device="R0603" value="10k"/>
+<part name="R9" library="dan" deviceset="R-US_" device="R0603" value="4.7k"/>
 <part name="P-2" library="dan" deviceset="-12V" device=""/>
 <part name="GND5" library="dan" deviceset="GND" device=""/>
@@
 <part name="C20" library="dan" deviceset="C-US" device="C0603" value="1u"/>
 <part name="C21" library="dan" deviceset="C-US" device="C0603" value="1u"/>
-<part name="D1" library="dan" deviceset="DUOLED5MM" device=""/>
 <part name="LED1" library="dan" deviceset="LED" device="5MM"/>
 <part name="LED2" library="dan" deviceset="LED" device="5MM"/>
@@
 <part name="GND31" library="dan" deviceset="GND" device=""/>
 <part name="R53" library="dan" deviceset="R-US_" device="R0603" value="1K"/>
+<part name="LED3" library="dan" deviceset="LED" device="5MM"/>
 </parts>
 <sheets>
 <sheet>
 <plain>
-<text x="45.72" y="40.64" size="1.778" layer="91">This is not confirmed.</text>
 <text x="10.16" y="-68.58" size="1.778" layer="91">Is this right?</text>
 <text x="-33.02" y="5.08" size="1.778" layer="91">Check these</text>
-<text x="-43.18" y="106.68" size="1.778" layer="91">Add LEDs!!!!</text>
 <text x="91.44" y="-50.8" size="1.778" layer="91">Changed to 10k</text>
 <text x="139.7" y="22.86" size="1.778" layer="91">Polarity backwards</text>
+<text x="231.14" y="10.16" size="1.778" layer="91">bicolor</text>
 </plain>
 <instances>
@@
 <instance part="C20" gate="G$1" x="-106.68" y="12.7" rot="R180"/>
 <instance part="C21" gate="G$1" x="-114.3" y="27.94"/>
-<instance part="D1" gate="1" x="226.06" y="15.24" rot="R270"/>
 <instance part="LED1" gate="G$1" x="132.08" y="50.8"/>
 <instance part="LED2" gate="G$1" x="48.26" y="2.54"/>
@@
 <instance part="GND31" gate="1" x="40.64" y="121.92"/>
 <instance part="R53" gate="G$1" x="48.26" y="127" rot="R270"/>
+<instance part="LED3" gate="G$1" x="226.06" y="12.7"/>
 </instances>
 <busses>
@@
 <wire x1="228.6" y1="30.48" x2="226.06" y2="30.48" width="0.1524" layer="91"/>
 <junction x="226.06" y="30.48"/>
-<pinref part="D1" gate="1" pin="C"/>
-<wire x1="226.06" y1="17.78" x2="226.06" y2="30.48" width="0.1524" layer="91"/>
+<wire x1="226.06" y1="15.24" x2="226.06" y2="30.48" width="0.1524" layer="91"/>
+<pinref part="LED3" gate="G$1" pin="A"/>
 </segment>
 </net>
@@
 <pinref part="ACVA" gate="G$1" pin="S"/>
 <wire x1="33.02" y1="-93.98" x2="30.48" y2="-93.98" width="0.1524" layer="91"/>
-</segment>
-</net>
-<net name="N$52" class="0">
-<segment>
-<pinref part="D1" gate="1" pin="AG"/>
-<wire x1="218.44" y1="15.24" x2="213.36" y2="15.24" width="0.1524" layer="91"/>
-<wire x1="213.36" y1="15.24" x2="213.36" y2="5.08" width="0.1524" layer="91"/>
-<wire x1="213.36" y1="5.08" x2="226.06" y2="5.08" width="0.1524" layer="91"/>
-<wire x1="226.06" y1="5.08" x2="236.22" y2="5.08" width="0.1524" layer="91"/>
-<wire x1="236.22" y1="5.08" x2="236.22" y2="15.24" width="0.1524" layer="91"/>
-<pinref part="D1" gate="1" pin="AR"/>
-<wire x1="236.22" y1="15.24" x2="233.68" y2="15.24" width="0.1524" layer="91"/>
-<pinref part="R48" gate="G$1" pin="1"/>
-<wire x1="226.06" y1="2.54" x2="226.06" y2="5.08" width="0.1524" layer="91"/>
-<junction x="226.06" y="5.08"/>
 </segment>
 </net>
@@
 </segment>
 </net>
+<net name="N$57" class="0">
+<segment>
+<pinref part="R48" gate="G$1" pin="1"/>
+<pinref part="LED3" gate="G$1" pin="C"/>
+<wire x1="226.06" y1="7.62" x2="226.06" y2="2.54" width="0.1524" layer="91"/>
+</segment>
+</net>
