File: keyboard/keyboard.brd (EAGLE design)
At the start: 297.2 x 60.6 mm, 49 parts

Commit message: made gerbers for vcf2
Parts:
- added D1, D10, D11, D12, D13, D14, D15, D16, D17, D18, D19, D2, D20, D21, D22, D23, D24, D25, D26, D27, D28, D29, D3, D30, D31, D32, D33, D34, D35, D36, D37, D38, D39, D4, D40, D41, D42, D43, D44, D45, D46, D5, D6, D7, D8, D9: MBR0520LT, dan:SOD123
- added R1, R10, R11, R2, R3, R4, R5, R6, R7, R8, R9: (no value), dan:R0603
- added SV1: (no value), dan:MA20-1
- added SV2, SV3, SV4: (no value), dan:MA04-1
- moved LED2 3.81 mm to (288.3, 47.0)
- moved LED3 3.81 mm to (7.62, 52.1)
- moved U$1 3.81 mm to (68.6, 16.5)
- moved U$10 3.81 mm to (151.1, 16.5)
- moved U$11 3.81 mm to (158.8, 33.0)
- moved U$12 3.81 mm to (167.6, 16.5)
- moved U$13 3.81 mm to (185.4, 16.5)
- moved U$14 3.81 mm to (193.0, 33.0)
- moved U$15 3.81 mm to (201.9, 16.5)
- moved U$16 3.81 mm to (209.6, 33.0)
- moved U$17 3.81 mm to (218.4, 16.5)
- moved U$18 3.81 mm to (234.9, 16.5)
- moved U$19 3.81 mm to (242.6, 33.0)
- moved U$2 3.81 mm to (76.2, 33.0)
- moved U$20 3.81 mm to (251.5, 16.5)
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Connections:
- new net COL1: D1.A, D15.A, D22.A, D29.A, D36.A, D43.A, D8.A, SV1.5
- new net COL2: D16.A, D2.A, D23.A, D30.A, D37.A, D44.A, D9.A, SV1.4
- new net COL3: D10.A, D17.A, D24.A, D3.A, D31.A, D38.A, D45.A, SV1.3
- new net COL4: D11.A, D18.A, D25.A, D32.A, D39.A, D4.A, D46.A, SV1.2
- new net COL5: D12.A, D19.A, D26.A, D33.A, D40.A, D5.A, SV1.1
- new net COL6: D13.A, D20.A, D27.A, D34.A, D41.A, D6.A
- new net COL7: D14.A, D21.A, D28.A, D35.A, D42.A, D7.A, SV2.3
- new net GND: R10.1, R11.1, R9.1, SV2.1, SV2.2, SV3.1, SV3.2, SV4.2, SV4.3
- new net LED1: R1.1, SV1.13
- new net LED2: SV1.14
- new net LED3: SV1.15
- new net LED4: R4.1, SV1.16
- new net LED5: R5.1, SV1.17
- new net LED6: R6.1, SV1.18
- new net LED7: R7.1, SV1.19
- new net LED8: R8.1, SV1.20
- new net N$1: D8.C, U$8.SW2
- new net N$10: D5.C, U$5.SW2
- new net N$11: D4.C, U$4.SW2
- new net N$12: D3.C, U$3.SW2
- new net N$13: D2.C, U$2.SW2
- new net N$14: D1.C, U$1.SW2
- new net N$15: D15.C, U$15.SW2
- new net N$16: D16.C, U$16.SW2
- new net N$17: D17.C, U$17.SW2
- new net N$18: D18.C, U$18.SW2
- new net N$19: D19.C, U$19.SW2
- new net N$2: D9.C, U$9.SW2
- new net N$20: D20.C, U$20.SW2
- new net N$21: D21.C, U$21.SW2
- new net N$22: D22.C
- new net N$23: D23.C
- new net N$24: D24.C
- new net N$25: D25.C
- new net N$26: D26.C
- new net N$27: D27.C, U$27.SW2
- new net N$28: D28.C, U$28.SW2
- new net N$29: D29.C, U$29.SW2
- new net N$3: D10.C, U$10.SW2
- new net N$30: D30.C, U$30.SW2
- new net N$31: D31.C, U$31.SW2
- new net N$32: D32.C, U$32.SW2
- new net N$33: D33.C, U$33.SW2
- new net N$34: D34.C, U$34.SW2
- new net N$35: D35.C, U$35.SW2
- new net N$36: D36.C, U$36.SW2
- new net N$37: D37.C, U$37.SW2
- new net N$38: D38.C, U$38.SW2
- new net N$39: D39.C, U$39.SW2
- new net N$4: D11.C, U$11.SW2
- new net N$40: D40.C, U$40.SW2
- new net N$41: D41.C, U$41.SW2
- new net N$42: D42.C, U$42.SW2
- new net N$43: D43.C, U$43.SW2
- new net N$44: D44.C, U$44.SW2
- new net N$45: D45.C, U$45.SW2
- new net N$46: D46.C, U$46.SW2
- new net N$48: LED1.K, R11.2
- new net N$49: R8.2, U$1.LED2, U$15.LED2, U$22.LED2, U$29.LED2, U$43.LED2, U$8.LED2
- new net N$5: D12.C, U$12.SW2
- new net N$50: R1.2, U$1.LED1, U$14.LED2, U$2.LED1, U$21.LED2, U$28.LED2, U$3.LED1, U$35.LED2, U$4.LED1, U$42.LED2, U$5.LED1, U$6.LED1, U$7.LED1
- new net N$51: R4.2, U$12.LED2, U$19.LED2, U$22.LED1, U$23.LED1, U$24.LED1, U$25.LED1, U$26.LED1, U$27.LED1, U$28.LED1, U$32.LED2, U$39.LED2, U$46.LED2, U$5.LED2
- new net N$52: R5.2, U$11.LED2, U$18.LED2, U$25.LED2, U$29.LED1, U$30.LED1, U$31.LED1, U$32.LED1, U$33.LED1, U$34.LED1, U$35.LED1, U$38.LED2, U$4.LED2, U$45.LED2
- new net N$53: R6.2, U$10.LED2, U$17.LED2, U$24.LED2, U$3.LED2, U$31.LED2, U$36.LED1, U$37.LED1, U$38.LED1, U$39.LED1, U$40.LED1, U$41.LED1, U$42.LED1, U$44.LED2
- new net N$54: LED2.K, R10.2
- new net N$55: LED3.K, R9.2
- new net N$58: LED1.A, SV3.3
- new net N$59: LED2.A, SV3.4
- new net N$6: D13.C, U$13.SW2
- new net N$60: LED3.A, SV4.1
- new net N$64: R7.2, U$16.LED2, U$2.LED2, U$23.LED2, U$30.LED2, U$37.LED2, U$43.LED1, U$44.LED1, U$45.LED1, U$46.LED1, U$9.LED2
- new net N$7: D14.C, U$14.SW2
- new net N$75: R2.2, U$10.LED1, U$11.LED1, U$13.LED1, U$14.LED1, U$20.LED2, U$27.LED2, U$34.LED2, U$41.LED2, U$7.LED2, U$8.LED1, U$9.LED1
- new net N$76: R3.2, U$13.LED2, U$15.LED1, U$16.LED1, U$17.LED1, U$18.LED1, U$19.LED1, U$20.LED1, U$21.LED1, U$26.LED2, U$40.LED2, U$6.LED2
- new net N$8: D7.C, U$7.SW2
- new net N$9: D6.C, U$6.SW2
- new net ROW1: SV1.6, U$1.SW1, U$2.SW1, U$3.SW1, U$4.SW1, U$5.SW1, U$6.SW1, U$7.SW1
- new net ROW2: SV1.7, U$10.SW1, U$11.SW1, U$12.SW1, U$13.SW1, U$14.SW1, U$8.SW1, U$9.SW1
- new net ROW3: SV1.8, U$15.SW1, U$16.SW1, U$17.SW1, U$18.SW1, U$19.SW1, U$20.SW1, U$21.SW1
- new net ROW4: SV1.9, U$22.SW1, U$23.SW1, U$24.SW1, U$25.SW1, U$26.SW1, U$27.SW1, U$28.SW1
- new net ROW5: SV1.10, U$29.SW1, U$30.SW1, U$31.SW1, U$32.SW1, U$33.SW1, U$34.SW1, U$35.SW1
- new net ROW6: SV1.11, U$36.SW1, U$37.SW1, U$38.SW1, U$39.SW1, U$40.SW1, U$41.SW1, U$42.SW1
- new net ROW7: SV1.12, U$43.SW1, U$44.SW1, U$45.SW1, U$46.SW1
Routing:
- added copper zone on layer 1, net GND
Other:
- board size 297.2 x 60.6 mm -> 297.2 x 61.9 mm
