File: vca/vca.brd (EAGLE design)
At the start: 43.2 x 219.7 mm, 59 parts, among them IC1 OPA4130U, IC2 OPA134D, Q1 BC847ALT1SMD, X1 2516-

Commit message: sent out vca again
Parts:
- moved SV6 1.27 mm to (39.4, 118.1)
- moved SV8 1.27 mm to (3.81, 118.1)
Routing:
- net N$5: track 50.3 -> 51.6 mm
- net N$32: track 93.0 -> 94.2 mm
- net N$31: track 94.8 -> 95.3 mm
Changed lines of the file:
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@@
 <layer number="19" name="Unrouted" color="6" fill="1" visible="yes" active="yes"/>
 <layer number="20" name="Dimension" color="15" fill="1" visible="yes" active="yes"/>
-<layer number="21" name="tPlace" color="7" fill="1" visible="yes" active="yes"/>
-<layer number="22" name="bPlace" color="7" fill="1" visible="yes" active="yes"/>
+<layer number="21" name="tPlace" color="7" fill="1" visible="no" active="yes"/>
+<layer number="22" name="bPlace" color="7" fill="1" visible="no" active="yes"/>
 <layer number="23" name="tOrigins" color="15" fill="1" visible="yes" active="yes"/>
 <layer number="24" name="bOrigins" color="15" fill="1" visible="yes" active="yes"/>
@@
 <attribute name="VALUE" x="37.719" y="9.525" size="1.27" layer="27" ratio="10" rot="R90"/>
 </element>
-<element name="SV6" library="dan" package="MA04-1" value="" x="39.37" y="119.38" smashed="yes" rot="R90">
-<attribute name="OC_NEWARK" value="unknown" x="39.37" y="119.38" size="1.778" layer="27" rot="R90" display="off"/>
-<attribute name="MPN" value="" x="39.37" y="119.38" size="1.778" layer="27" rot="R90" display="off"/>
-<attribute name="MF" value="" x="39.37" y="119.38" size="1.778" layer="27" rot="R90" display="off"/>
-<attribute name="OC_FARNELL" value="unknown" x="39.37" y="119.38" size="1.778" layer="27" rot="R90" display="off"/>
-<attribute name="NAME" x="35.941" y="121.92" size="1.27" layer="21" font="vector" ratio="15" rot="R270"/>
-<attribute name="VALUE" x="37.719" y="120.015" size="1.27" layer="27" ratio="10" rot="R90"/>
+<element name="SV6" library="dan" package="MA04-1" value="" x="39.37" y="118.11" smashed="yes" rot="R90">
+<attribute name="OC_NEWARK" value="unknown" x="39.37" y="118.11" size="1.778" layer="27" rot="R90" display="off"/>
+<attribute name="MPN" value="" x="39.37" y="118.11" size="1.778" layer="27" rot="R90" display="off"/>
+<attribute name="MF" value="" x="39.37" y="118.11" size="1.778" layer="27" rot="R90" display="off"/>
+<attribute name="OC_FARNELL" value="unknown" x="39.37" y="118.11" size="1.778" layer="27" rot="R90" display="off"/>
+<attribute name="NAME" x="35.941" y="120.65" size="1.27" layer="21" font="vector" ratio="15" rot="R270"/>
+<attribute name="VALUE" x="37.719" y="118.745" size="1.27" layer="27" ratio="10" rot="R90"/>
 </element>
 <element name="SV7" library="dan" package="MA04-1" value="" x="3.81" y="8.89" smashed="yes" rot="R90">
@@
 <attribute name="VALUE" x="2.159" y="9.525" size="1.27" layer="27" ratio="10" rot="R90"/>
 </element>
-<element name="SV8" library="dan" package="MA04-1" value="" x="3.81" y="119.38" smashed="yes" rot="R90">
-<attribute name="OC_NEWARK" value="unknown" x="3.81" y="119.38" size="1.778" layer="27" rot="R90" display="off"/>
-<attribute name="MPN" value="" x="3.81" y="119.38" size="1.778" layer="27" rot="R90" display="off"/>
-<attribute name="MF" value="" x="3.81" y="119.38" size="1.778" layer="27" rot="R90" display="off"/>
-<attribute name="OC_FARNELL" value="unknown" x="3.81" y="119.38" size="1.778" layer="27" rot="R90" display="off"/>
-<attribute name="NAME" x="7.239" y="118.11" size="1.27" layer="21" font="vector" ratio="15" rot="R90"/>
-<attribute name="VALUE" x="2.159" y="120.015" size="1.27" layer="27" ratio="10" rot="R90"/>
+<element name="SV8" library="dan" package="MA04-1" value="" x="3.81" y="118.11" smashed="yes" rot="R90">
+<attribute name="OC_NEWARK" value="unknown" x="3.81" y="118.11" size="1.778" layer="27" rot="R90" display="off"/>
+<attribute name="MPN" value="" x="3.81" y="118.11" size="1.778" layer="27" rot="R90" display="off"/>
+<attribute name="MF" value="" x="3.81" y="118.11" size="1.778" layer="27" rot="R90" display="off"/>
+<attribute name="OC_FARNELL" value="unknown" x="3.81" y="118.11" size="1.778" layer="27" rot="R90" display="off"/>
+<attribute name="NAME" x="7.239" y="116.84" size="1.27" layer="21" font="vector" ratio="15" rot="R90"/>
+<attribute name="VALUE" x="2.159" y="118.745" size="1.27" layer="27" ratio="10" rot="R90"/>
 </element>
 <element name="C1" library="dan" package="C0603" value="2.2u" x="8.89" y="215.9" smashed="yes" rot="R180">
@@
 <wire x1="22.86" y1="173.99" x2="21.59" y2="175.26" width="0.6096" layer="1"/>
 <wire x1="21.59" y1="175.26" x2="21.59" y2="180.34" width="0.6096" layer="1"/>
-<wire x1="34.29" y1="115.57" x2="39.37" y2="115.57" width="0.6096" layer="16"/>
+<wire x1="35.56" y1="114.3" x2="39.37" y2="114.3" width="0.6096" layer="16"/>
 <wire x1="22.86" y1="147.32" x2="22.86" y2="129.54" width="0.6096" layer="1"/>
 <wire x1="22.86" y1="129.54" x2="27.94" y2="124.46" width="0.6096" layer="1"/>
 <wire x1="27.94" y1="124.46" x2="29.21" y2="124.46" width="0.6096" layer="1"/>
-<wire x1="29.21" y1="124.46" x2="33.02" y2="120.65" width="0.6096" layer="1"/>
-<wire x1="33.02" y1="120.65" x2="33.02" y2="116.84" width="0.6096" layer="1"/>
-<wire x1="33.02" y1="116.84" x2="34.29" y2="115.57" width="0.6096" layer="1"/>
-<via x="34.29" y="115.57" extent="1-16" drill="0.7"/>
+<wire x1="29.21" y1="124.46" x2="35.56" y2="118.11" width="0.6096" layer="1"/>
+<wire x1="35.56" y1="118.11" x2="35.56" y2="114.3" width="0.6096" layer="1"/>
+<via x="35.56" y="114.3" extent="1-16" drill="0.7"/>
 </signal>
 <signal name="N$33">
@@
 <wire x1="31.75" y1="143.51" x2="22.86" y2="143.51" width="0.6096" layer="16"/>
 <wire x1="22.86" y1="143.51" x2="16.51" y2="132.08" width="0.6096" layer="16"/>
-<wire x1="3.81" y1="115.57" x2="6.35" y2="115.57" width="0.6096" layer="1"/>
-<wire x1="6.35" y1="115.57" x2="7.62" y2="116.84" width="0.6096" layer="1"/>
-<wire x1="7.62" y1="116.84" x2="7.62" y2="119.38" width="0.6096" layer="1"/>
-<wire x1="7.62" y1="119.38" x2="6.35" y2="120.65" width="0.6096" layer="1"/>
-<wire x1="6.35" y1="120.65" x2="6.35" y2="129.54" width="0.6096" layer="1"/>
+<wire x1="3.81" y1="114.3" x2="6.35" y2="114.3" width="0.6096" layer="1"/>
+<wire x1="6.35" y1="114.3" x2="7.62" y2="115.57" width="0.6096" layer="1"/>
+<wire x1="7.62" y1="115.57" x2="7.62" y2="118.11" width="0.6096" layer="1"/>
+<wire x1="7.62" y1="118.11" x2="6.35" y2="119.38" width="0.6096" layer="1"/>
+<wire x1="6.35" y1="119.38" x2="6.35" y2="129.54" width="0.6096" layer="1"/>
 <wire x1="6.35" y1="129.54" x2="7.62" y2="130.81" width="0.6096" layer="1"/>
 <via x="7.62" y="130.81" extent="1-16" drill="0.7"/>
@@
 <wire x1="20.32" y1="132.08" x2="39.37" y2="132.08" width="0.6096" layer="16"/>
 <via x="39.37" y="132.08" extent="1-16" drill="0.7"/>
-<wire x1="39.37" y1="132.08" x2="39.37" y2="123.19" width="0.6096" layer="1"/>
+<wire x1="39.37" y1="132.08" x2="39.37" y2="121.92" width="0.6096" layer="1"/>
 <via x="19.05" y="175.26" extent="1-16" drill="0.7"/>
 <wire x1="20.32" y1="132.08" x2="20.32" y2="146.05" width="0.6096" layer="1"/>

Commit message: progress..
Parts:
- moved R20 1.27 mm to (6.35, 182.9)
- moved AMP 1.27 mm to (8.89, 193.0)
- moved IN2G 1.27 mm to (8.89, 166.4)
- moved R19 1.27 mm to (11.4, 182.9)
- moved CVA 1.27 mm to (34.3, 193.0)
- moved IN1G 1.27 mm to (34.3, 166.4)
Routing:
- net N$41: track 93.9 -> 89.6 mm
- net N$37: track 100.8 -> 104.3 mm
- net N$19: track 98.2 -> 101.0 mm
- net N$40: track 78.0 -> 79.8 mm
- net +12V: track 196.1 -> 197.3 mm
- net N$21: track 93.1 -> 94.4 mm
- net N$27: track 51.9 -> 50.7 mm
- net N$32: track 94.2 -> 95.4 mm
- net N$31: track 95.3 -> 96.4 mm
- net N$26: track 65.2 -> 66.2 mm
- net N$25: track 38.8 -> 38.3 mm
