File: vcf2/vcf2.sch (EAGLE design)
At the start: 115 parts, among them IC1 OPA4130U, IC2 OPA4130U, IC3 OPA4130U, IC4 OPA4130U, IC5 OPA4130U, Q7 BC847ASMD

Commit message: vcf2 changes
Connections:
- new net N$90: R47.2, SV8.4
- net GND: no longer SV7.1, SV8.1
- net N$24: now also SV7.3; no longer SV7.4
- net N$33: now also SV7.2; no longer SV7.3
- net N$50: now also SV8.1; no longer SV8.2
- net N$73: now also SV7.4; no longer R47.2
- net N$79: now also SV8.2; no longer SV8.3
- net N$80: now also SV8.3; no longer SV8.4
- net N$81: now also SV7.1; no longer SV7.2
Other:
- moved on the sheet: FREQ, MAXFREQ, R44, R47, R48
Changed lines of the file:
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@@
 <part name="P-10" library="dan" deviceset="-12V" device=""/>
 <part name="GND31" library="dan" deviceset="GND" device=""/>
-<part name="GND32" library="dan" deviceset="GND" device=""/>
-<part name="GND33" library="dan" deviceset="GND" device=""/>
 <part name="GND34" library="dan" deviceset="GND" device=""/>
 <part name="GND35" library="dan" deviceset="GND" device=""/>
@@
 <instance part="GND20" gate="1" x="269.24" y="116.84"/>
 <instance part="GND21" gate="1" x="271.78" y="149.86"/>
-<instance part="FREQ" gate="G$1" x="-73.66" y="-88.9" rot="MR180"/>
-<instance part="P-7" gate="1" x="-73.66" y="-114.3"/>
-<instance part="P+9" gate="1" x="-58.42" y="-58.42"/>
-<instance part="R44" gate="G$1" x="-60.96" y="-88.9"/>
+<instance part="FREQ" gate="G$1" x="-73.66" y="-91.44" rot="MR180"/>
+<instance part="P-7" gate="1" x="-73.66" y="-116.84"/>
+<instance part="P+9" gate="1" x="-116.84" y="20.32"/>
+<instance part="R44" gate="G$1" x="-60.96" y="-91.44"/>
 <instance part="GAIN1" gate="G$1" x="-12.7" y="68.58" rot="MR0"/>
 <instance part="C5" gate="G$1" x="-20.32" y="38.1" rot="R270"/>
@@
 <instance part="R45" gate="G$1" x="220.98" y="66.04" rot="R180"/>
 <instance part="R46" gate="G$1" x="167.64" y="193.04" rot="R180"/>
-<instance part="R47" gate="G$1" x="-73.66" y="-73.66" rot="R90"/>
-<instance part="R48" gate="G$1" x="-73.66" y="-104.14" rot="R90"/>
+<instance part="R47" gate="G$1" x="-73.66" y="-76.2" rot="R90"/>
+<instance part="R48" gate="G$1" x="-73.66" y="-106.68" rot="R90"/>
 <instance part="R49" gate="G$1" x="20.32" y="76.2" rot="R90"/>
 <instance part="P+11" gate="1" x="-10.16" y="12.7"/>
@@
 <instance part="R9" gate="G$1" x="-45.72" y="177.8" rot="R180"/>
 <instance part="R51" gate="G$1" x="-45.72" y="154.94" rot="R180"/>
-<instance part="MAXFREQ" gate="G$1" x="-58.42" y="-71.12"/>
+<instance part="MAXFREQ" gate="G$1" x="-116.84" y="7.62"/>
 <instance part="MAXRES" gate="G$1" x="139.7" y="76.2"/>
 <instance part="U$1" gate="G$1" x="35.56" y="38.1"/>
@@
 <instance part="P-10" gate="1" x="-45.72" y="96.52"/>
 <instance part="GND31" gate="1" x="-55.88" y="96.52"/>
-<instance part="GND32" gate="1" x="-48.26" y="-101.6"/>
-<instance part="GND33" gate="1" x="-116.84" y="-20.32"/>
 <instance part="GND34" gate="1" x="223.52" y="124.46"/>
 <instance part="GND35" gate="1" x="269.24" y="124.46"/>
@@
 </segment>
 <segment>
-<pinref part="GND32" gate="1" pin="GND"/>
-<wire x1="-48.26" y1="-99.06" x2="-48.26" y2="-96.52" width="0.1524" layer="91"/>
-<pinref part="SV8" gate="1" pin="1"/>
-<wire x1="-48.26" y1="-96.52" x2="-45.72" y2="-96.52" width="0.1524" layer="91"/>
-</segment>
-<segment>
-<pinref part="SV7" gate="1" pin="1"/>
-<wire x1="-119.38" y1="-10.16" x2="-116.84" y2="-10.16" width="0.1524" layer="91"/>
-<wire x1="-116.84" y1="-10.16" x2="-116.84" y2="-17.78" width="0.1524" layer="91"/>
-<pinref part="GND33" gate="1" pin="GND"/>
-</segment>
-<segment>
 <pinref part="SV12" gate="1" pin="3"/>
 <pinref part="GND34" gate="1" pin="GND"/>
@@
 <pinref part="MAXFREQ" gate="G$1" pin="E"/>
 <pinref part="P+9" gate="1" pin="+12V"/>
-<wire x1="-58.42" y1="-60.96" x2="-58.42" y2="-63.5" width="0.1524" layer="91"/>
+<wire x1="-116.84" y1="17.78" x2="-116.84" y2="15.24" width="0.1524" layer="91"/>
 </segment>
 <segment>
@@
 <pinref part="P-7" gate="1" pin="-12V"/>
 <pinref part="R48" gate="G$1" pin="1"/>
-<wire x1="-73.66" y1="-111.76" x2="-73.66" y2="-109.22" width="0.1524" layer="91"/>
+<wire x1="-73.66" y1="-114.3" x2="-73.66" y2="-111.76" width="0.1524" layer="91"/>
 </segment>
 <segment>
@@
 <pinref part="FREQ" gate="G$1" pin="A"/>
 <pinref part="R47" gate="G$1" pin="1"/>
-<wire x1="-73.66" y1="-81.28" x2="-73.66" y2="-78.74" width="0.1524" layer="91"/>
+<wire x1="-73.66" y1="-83.82" x2="-73.66" y2="-81.28" width="0.1524" layer="91"/>
 </segment>
 </net>
@@
 <pinref part="FREQ" gate="G$1" pin="S"/>
 <pinref part="R44" gate="G$1" pin="1"/>
-<wire x1="-68.58" y1="-88.9" x2="-66.04" y2="-88.9" width="0.1524" layer="91"/>
+<wire x1="-68.58" y1="-91.44" x2="-66.04" y2="-91.44" width="0.1524" layer="91"/>
 </segment>
 </net>
@@
 <pinref part="FREQ" gate="G$1" pin="E"/>
 <pinref part="R48" gate="G$1" pin="2"/>
-<wire x1="-73.66" y1="-96.52" x2="-73.66" y2="-99.06" width="0.1524" layer="91"/>
+<wire x1="-73.66" y1="-99.06" x2="-73.66" y2="-101.6" width="0.1524" layer="91"/>
 </segment>
 </net>
@@
 <pinref part="MODAMT" gate="G$1" pin="S"/>
 <wire x1="-53.34" y1="-109.22" x2="-55.88" y2="-109.22" width="0.1524" layer="91"/>
-<pinref part="SV8" gate="1" pin="2"/>
-<wire x1="-45.72" y1="-93.98" x2="-53.34" y2="-93.98" width="0.1524" layer="91"/>
-<wire x1="-53.34" y1="-93.98" x2="-53.34" y2="-109.22" width="0.1524" layer="91"/>
+<wire x1="-53.34" y1="-96.52" x2="-53.34" y2="-109.22" width="0.1524" layer="91"/>
+<pinref part="SV8" gate="1" pin="1"/>
+<wire x1="-45.72" y1="-96.52" x2="-53.34" y2="-96.52" width="0.1524" layer="91"/>
 </segment>
 </net>
@@
 <wire x1="-134.62" y1="-15.24" x2="-134.62" y2="-17.78" width="0.1524" layer="91"/>
 <wire x1="-134.62" y1="-15.24" x2="-109.22" y2="-15.24" width="0.1524" layer="91"/>
-<wire x1="-109.22" y1="-15.24" x2="-109.22" y2="-5.08" width="0.1524" layer="91"/>
-<pinref part="SV7" gate="1" pin="3"/>
-<wire x1="-109.22" y1="-5.08" x2="-119.38" y2="-5.08" width="0.1524" layer="91"/>
+<wire x1="-109.22" y1="-15.24" x2="-109.22" y2="-7.62" width="0.1524" layer="91"/>
 <junction x="-134.62" y="-15.24"/>
+<pinref part="SV7" gate="1" pin="2"/>
+<wire x1="-109.22" y1="-7.62" x2="-119.38" y2="-7.62" width="0.1524" layer="91"/>
 </segment>
 </net>
@@
 <net name="N$73" class="0">
 <segment>
-<wire x1="-50.8" y1="-71.12" x2="-50.8" y2="-81.28" width="0.1524" layer="91"/>
-<wire x1="-50.8" y1="-81.28" x2="-58.42" y2="-81.28" width="0.1524" layer="91"/>
+<wire x1="-109.22" y1="7.62" x2="-109.22" y2="-2.54" width="0.1524" layer="91"/>
+<wire x1="-109.22" y1="-2.54" x2="-116.84" y2="-2.54" width="0.1524" layer="91"/>
+<pinref part="MAXFREQ" gate="G$1" pin="S"/>
+<wire x1="-116.84" y1="-2.54" x2="-119.38" y2="-2.54" width="0.1524" layer="91"/>
+<wire x1="-111.76" y1="7.62" x2="-109.22" y2="7.62" width="0.1524" layer="91"/>
+<pinref part="SV7" gate="1" pin="4"/>
 <pinref part="MAXFREQ" gate="G$1" pin="A"/>
-<wire x1="-58.42" y1="-81.28" x2="-58.42" y2="-78.74" width="0.1524" layer="91"/>
-<wire x1="-58.42" y1="-81.28" x2="-68.58" y2="-81.28" width="0.1524" layer="91"/>
-<wire x1="-68.58" y1="-81.28" x2="-68.58" y2="-66.04" width="0.1524" layer="91"/>
-<pinref part="R47" gate="G$1" pin="2"/>
-<wire x1="-68.58" y1="-66.04" x2="-73.66" y2="-66.04" width="0.1524" layer="91"/>
-<wire x1="-73.66" y1="-66.04" x2="-73.66" y2="-68.58" width="0.1524" layer="91"/>
-<junction x="-58.42" y="-81.28"/>
-<pinref part="MAXFREQ" gate="G$1" pin="S"/>
-<wire x1="-53.34" y1="-71.12" x2="-50.8" y2="-71.12" width="0.1524" layer="91"/>
+<wire x1="-116.84" y1="0" x2="-116.84" y2="-2.54" width="0.1524" layer="91"/>
+<junction x="-116.84" y="-2.54"/>
 </segment>
 </net>
@@
 <pinref part="IC5" gate="B" pin="+IN"/>
 <wire x1="-53.34" y1="-30.48" x2="-91.44" y2="-30.48" width="0.1524" layer="91"/>
-<wire x1="-91.44" y1="-30.48" x2="-91.44" y2="-2.54" width="0.1524" layer="91"/>
-<pinref part="SV7" gate="1" pin="4"/>
-<wire x1="-91.44" y1="-2.54" x2="-119.38" y2="-2.54" width="0.1524" layer="91"/>
+<wire x1="-91.44" y1="-30.48" x2="-91.44" y2="-5.08" width="0.1524" layer="91"/>
+<pinref part="SV7" gate="1" pin="3"/>
+<wire x1="-91.44" y1="-5.08" x2="-119.38" y2="-5.08" width="0.1524" layer="91"/>
 </segment>
 </net>
@@
 <segment>
 <pinref part="MODAMT" gate="G$1" pin="E"/>
-<pinref part="SV8" gate="1" pin="3"/>
-<wire x1="-45.72" y1="-91.44" x2="-60.96" y2="-91.44" width="0.1524" layer="91"/>
-<wire x1="-60.96" y1="-91.44" x2="-60.96" y2="-101.6" width="0.1524" layer="91"/>
-</segment>
-</net>
-<net name="N$80" class="0">
-<segment>
-<pinref part="R44" gate="G$1" pin="2"/>
-<pinref part="SV8" gate="1" pin="4"/>
-<wire x1="-55.88" y1="-88.9" x2="-45.72" y2="-88.9" width="0.1524" layer="91"/>
+<wire x1="-60.96" y1="-93.98" x2="-60.96" y2="-101.6" width="0.1524" layer="91"/>
+<pinref part="SV8" gate="1" pin="2"/>
+<wire x1="-45.72" y1="-93.98" x2="-60.96" y2="-93.98" width="0.1524" layer="91"/>
 </segment>
 </net>
 <net name="N$81" class="0">
 <segment>
-<pinref part="SV7" gate="1" pin="2"/>
-<wire x1="-119.38" y1="-7.62" x2="-111.76" y2="-7.62" width="0.1524" layer="91"/>
-<wire x1="-111.76" y1="-7.62" x2="-111.76" y2="-33.02" width="0.1524" layer="91"/>
+<wire x1="-111.76" y1="-10.16" x2="-111.76" y2="-33.02" width="0.1524" layer="91"/>
 <pinref part="IC1" gate="C" pin="+IN"/>
 <wire x1="-111.76" y1="-33.02" x2="-109.22" y2="-33.02" width="0.1524" layer="91"/>
+<pinref part="SV7" gate="1" pin="1"/>
+<wire x1="-111.76" y1="-10.16" x2="-119.38" y2="-10.16" width="0.1524" layer="91"/>
 </segment>
 </net>
@@
 </segment>
 </net>
+<net name="N$80" class="0">
+<segment>
+<pinref part="SV8" gate="1" pin="3"/>
+<pinref part="R44" gate="G$1" pin="2"/>
+<wire x1="-45.72" y1="-91.44" x2="-55.88" y2="-91.44" width="0.1524" layer="91"/>
+</segment>
+</net>
+<net name="N$90" class="0">
+<segment>
+<pinref part="R47" gate="G$1" pin="2"/>
+<wire x1="-73.66" y1="-68.58" x2="-73.66" y2="-71.12" width="0.1524" layer="91"/>
+<wire x1="-68.58" y1="-88.9" x2="-68.58" y2="-68.58" width="0.1524" layer="91"/>
+<wire x1="-68.58" y1="-68.58" x2="-73.66" y2="-68.58" width="0.1524" layer="91"/>
+<pinref part="SV8" gate="1" pin="4"/>
+<wire x1="-45.72" y1="-88.9" x2="-68.58" y2="-88.9" width="0.1524" layer="91"/>
+</segment>
+</net>

Commit message: made gerbers for vcf2
Connections:
- net N$86: now also GAIN.S
Changed lines of the file:
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@@
 <wire x1="-43.18" y1="81.28" x2="-22.86" y2="81.28" width="0.1524" layer="91"/>
 <wire x1="-22.86" y1="81.28" x2="-22.86" y2="96.52" width="0.1524" layer="91"/>
-<wire x1="-22.86" y1="96.52" x2="-15.24" y2="96.52" width="0.1524" layer="91"/>
+<wire x1="-22.86" y1="96.52" x2="-17.78" y2="96.52" width="0.1524" layer="91"/>
+<pinref part="GAIN" gate="G$1" pin="S"/>
 </segment>
 </net>

Commit message: progress..
Parts:
- R19, R20: value 47k -> 22k
Changed lines of the file:
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@@
 <part name="Q" library="dan" deviceset="US-EVU" device="F2J" value="10K"/>
 <part name="R18" library="dan" deviceset="R-US_" device="R0603" value="1k"/>
-<part name="R19" library="dan" deviceset="R-US_" device="R0603" value="47k"/>
-<part name="R20" library="dan" deviceset="R-US_" device="R0603" value="47k"/>
+<part name="R19" library="dan" deviceset="R-US_" device="R0603" value="22k"/>
+<part name="R20" library="dan" deviceset="R-US_" device="R0603" value="22k"/>
 <part name="GND6" library="dan" deviceset="GND" device=""/>
 <part name="GAIN" library="dan" deviceset="US-EVU" device="F2J" value="10K"/>
