File: vco2/vco_main.brd (EAGLE design)
At the start: 94.9 x 107.9 mm, 115 parts, among them IC1 OPA4130U, IC2 LM13700M, IC3 OPA4130U, IC4 OPA4130U, Q1 MMBFJ3

Commit message: more work on vco2
Parts:
- moved SV11 113.1 mm to (77.5, 59.7)
- moved SV13 110.7 mm to (77.5, 76.2)
- moved SV9 106.7 mm to (74.9, 7.62)
- moved SV1 83.9 mm to (5.08, 8.89)
- moved SV3 83.9 mm to (5.08, 25.4)
- moved SV5 83.9 mm to (5.08, 49.5)
- moved SV7 83.9 mm to (5.08, 73.7)
- moved SCALE 41.3 mm to (74.9, 22.9)
- moved R49 41.0 mm to (55.9, 15.2)
- moved R23 40.9 mm to (52.1, 15.2)
- moved C4 40.9 mm to (49.5, 29.2)
- moved R22 40.9 mm to (49.5, 15.2)
- moved R36 40.9 mm to (45.7, 16.5)
- moved R46 40.9 mm to (40.6, 16.5)
- moved SAWTRIM 39.1 mm to (74.9, 30.5)
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
Commit message: progress..
Parts:
- removed C4: 1u, dan:C0603
- removed LED1: (no value), dan:LED5MM
- removed Q1: MMBFJ3, dan:SOT23
- removed R44, R49: 1K, dan:R0603
- removed R45, R51: 10K, dan:R0603
- removed R47: 4.7K, dan:R0603
- removed SIN: PJ301BM, dan:PJ301BM
- removed SINTRIM: (no value), dan:B64Y
- removed U$4, U$5: 1N4148W, dan:SOD123
- added PW, PWM: 10K, dan:EVUFXJ
- added PWIN, PWOUT: PJ301BM, dan:PJ301BM
- R24: value 1Meg -> 1k
- R34: value 4.7K -> 10K
- R35: value 10K -> 1k
- R38: value 10K -> 1K
- R39: value 10K -> 10k
- R40: value 1Meg -> 10k
- R41: value 1Meg -> 10K
- R42, R43: value 110 -> 1K
- moved R15 89.5 mm to (78.7, 82.5)
- moved R16 89.5 mm to (73.7, 82.5)
- moved SV10 74.0 mm to (129.5, 78.7)
- moved SV9 72.2 mm to (62.2, 78.7)
- moved SV13 68.1 mm to (61.0, 10.2)
- moved R14 63.6 mm to (104.1, 82.5)
- moved R17 63.6 mm to (99.1, 82.5)
- moved SV3 59.5 mm to (62.2, 41.9), turned to 270 degrees
- moved SYNC 57.9 mm to (120.7, 74.9)
- moved R42 56.6 mm to (94.0, 16.5), turned to 0 degrees
- moved COARSE 55.9 mm to (76.2, 95.2)
- moved S1 54.6 mm to (120.7, 94.0)
- moved R46 53.6 mm to (72.4, 59.7)
- moved SQUARE 52.1 mm to (80.0, 8.89)
- moved TRIOUT 52.1 mm to (80.0, 25.4)
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Connections:
- removed net N$37 (its old number): Q1.3, R40.1, R41.2, U$4.A, U$5.A
- removed net N$52 (its old number): IC4.8, IC4.9, SV11.3
- removed net N$59: IC4.10, R51.2
- removed net N$70: LED1.K, SV12.3
- new net N$33: PWOUT.P$3, R42.2
- new net N$71: IC3.12, SV3.2
- new net N$72: PWIN.P$3, PWM.2
- net +12V: now also R24.2
- net -12V: now also R35.1
- net GND: now also PWIN.P$1, PWIN.P$4, PWM.1, PWOUT.P$1, PWOUT.P$4, R41.2, SV11.3, SV12.3; no longer IC3.10, IC3.12, R24.1, R41.1, R42.1, R45.2, R47.2, SIN.P$1, SIN.P$4, SINTRIM.E, SV3.2, SV4.2, U$4.C
- net N$1: now also IC3.14, R34.1; no longer LED1.A, R47.1
- net N$34: now also IC3.10, R34.2, R41.1; no longer IC3.9, R34.1, R35.2
- net N$35: now also R43.2, SQUARE.P$3; no longer C4.1, SINTRIM.A
- net N$36: now also IC3.9, SV3.3; no longer R34.2, R49.1
- net N$38: now also R40.2, SV4.2; no longer IC3.13, R38.1
- net N$39: now also PW.2; no longer SINTRIM.S
- net N$40: now also IC4.8, IC4.9, SV7.3; no longer R44.2, R45.1, SV3.3
- net N$41: now also PW.1, R24.1; no longer IC3.14, R38.2, R40.2, R43.2, U$5.C
- net N$43: now also PW.3, R35.2; no longer Q1.1, R42.2, R44.1
- net N$44: now also PWM.3, R40.1; no longer Q1.2, R43.1
- net N$57: now also R38.2; no longer R24.2, R35.1
- net N$61: now also R42.1; no longer SIN.P$3
- net N$65: now also R43.1; no longer SQUARE.P$3
- net N$9: now also IC4.10, R38.1; no longer R49.2, SV7.3
- net TRI: now also IC3.13; no longer C4.2, R51.1
Routing:
- added copper zone on layer 1, net GND
Other:
- board size 94.9 x 107.9 mm -> 133 x 104.1 mm
- board text removed: "expmod"
- board text removed: "linmod"
- board text removed: "saw"
- board text removed: "sine"
- board text removed: "square"
- board text removed: "sync"
- board text removed: "triangle"
- board text removed: "vperoct"
