File: vco2/vco_main.sch (EAGLE design)
At the start: 115 parts, among them IC1 OPA4130U, IC2 LM13700M, IC3 OPA4130U, IC4 OPA4130U, Q1 MMBFJ3

Commit message: progress..
Parts:
- removed C4: 1u, dan:C-USC0603
- removed LED1: (no value), dan:LED5MM
- removed Q1: MMBFJ3, dan:MMBFJ3
- removed R44, R49: 1K, dan:R-US_R0603
- removed R45, R51: 10K, dan:R-US_R0603
- removed R47: 4.7K, dan:R-US_R0603
- removed SIN: PJ301BM, dan:PJ301BM
- removed SINTRIM: (no value), dan:TRIM_US-B64Y
- removed U$4, U$5: 1N4148W, dan:1N4148W
- added PW, PWM: 10K, dan:US-EVUF2J
- added PWIN, PWOUT: PJ301BM, dan:PJ301BM
- R24: value 1Meg -> 1k
- R34: value 4.7K -> 10K
- R35: value 10K -> 1k
- R38: value 10K -> 1K
- R39: value 10K -> 10k
- R40: value 1Meg -> 10k
- R41: value 1Meg -> 10K
- R42, R43: value 110 -> 1K
Connections:
- removed net N$37 (its old number): Q1.G, R40.1, R41.2, U$4.A, U$5.A
- removed net N$52 (its old number): IC4C.-IN, IC4C.OUT, SV11.3
- removed net N$59: IC4C.+IN, R51.2
- removed net N$70: LED1.C, SV12.3
- new net N$33: PWOUT.P$3, R42.2
- new net N$71: IC3D.+IN, SV3.2
- new net N$72: PWIN.P$3, PWM.S
- net +12V: now also R24.2
- net -12V: now also R35.1
- net GND: now also PWIN.P$1, PWIN.P$4, PWM.A, PWOUT.P$1, PWOUT.P$4, R41.2, SV11.3, SV12.3; no longer IC3C.+IN, IC3D.+IN, R24.1, R41.1, R42.1, R45.2, R47.2, SIN.P$1, SIN.P$4, SINTRIM.E, SV3.2, SV4.2, U$4.C
- net N$1: now also IC3D.OUT, R34.1; no longer LED1.A, R47.1
- net N$34: now also IC3C.+IN, R34.2, R41.1; no longer IC3C.-IN, R34.1, R35.2
- net N$35: now also R43.2, SQUARE.P$3; no longer C4.1, SINTRIM.A
- net N$36: now also IC3C.-IN, SV3.3; no longer R34.2, R49.1
- net N$38: now also R40.2, SV4.2; no longer IC3D.-IN, R38.1
- net N$39: now also PW.S; no longer SINTRIM.S
- net N$40: now also IC4C.-IN, IC4C.OUT, SV7.3; no longer R44.2, R45.1, SV3.3
- net N$41: now also PW.A, R24.1; no longer IC3D.OUT, R38.2, R40.2, R43.2, U$5.C
- net N$43: now also PW.E, R35.2; no longer Q1.D, R42.2, R44.1
- net N$44: now also PWM.E, R40.1; no longer Q1.S, R43.1
- net N$57: now also R38.2; no longer R24.2, R35.1
- net N$61: now also R42.1; no longer SIN.P$3
- net N$65: now also R43.1; no longer SQUARE.P$3
- net N$9: now also IC4C.+IN, R38.1; no longer R49.2, SV7.3
- net TRI: now also IC3D.-IN; no longer C4.2, R51.1
Other:
- note removed: "Verify location of sync input"
- moved on the sheet: C10, C11, C12, C13, C14, C15, C16, C17, C18, C19, C2, C3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
